Commit message: add euler comand

File: cyclonedds_ws/src/urdf/go2.urdf (robot description, URDF)
Before this commit: robot go2, 33 links, 32 joints
Links:
- link FL_calf: geometry collision cylinder length=0.12 radius=0.012; visual mesh filename=/home/user/unitree_ros2/cyclonedds_ws/src/dae/calf.dae
- link FL_foot: geometry collision sphere radius=0.022; visual mesh filename=/home/user/unitree_ros2/cyclonedds_ws/src/dae/foot.dae
- link FL_hip: geometry collision cylinder length=0.04 radius=0.046; visual mesh filename=/home/user/unitree_ros2/cyclonedds_ws/src/dae/hip.dae
- link FL_thigh: geometry collision box size=0.213 0.0245 0.034; visual mesh filename=/home/user/unitree_ros2/cyclonedds_ws/src/dae/thigh.dae
- link FR_calf: geometry collision cylinder length=0.12 radius=0.013; visual mesh filename=/home/user/unitree_ros2/cyclonedds_ws/src/dae/calf_mirror.d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
- link FR_foot: geometry collision sphere radius=0.022; visual mesh filename=/home/user/unitree_ros2/cyclonedds_ws/src/dae/foot.dae
- link FR_hip: geometry collision cylinder length=0.04 radius=0.046; visual mesh filename=/home/user/unitree_ros2/cyclonedds_ws/src/dae/hip.dae
- link FR_thigh: geometry collision box size=0.213 0.0245 0.034; visual mesh filename=/home/user/unitree_ros2/cyclonedds_ws/src/dae/thigh_mirror.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
- link RL_calf: geometry collision cylinder length=0.12 radius=0.013; visual mesh filename=/home/user/unitree_ros2/cyclonedds_ws/src/dae/calf.dae
- link RL_foot: geometry collision sphere radius=0.022; visual mesh filename=/home/user/unitree_ros2/cyclonedds_ws/src/dae/foot.dae
- link RL_hip: geometry collision cylinder length=0.04 radius=0.046; visual mesh filename=/home/user/unitree_ros2/cyclonedds_ws/src/dae/hip.dae
- link RL_thigh: geometry collision box size=0.213 0.0245 0.034; visual mesh filename=/home/user/unitree_ros2/cyclonedds_ws/src/dae/thigh.dae
- link RR_calf: geometry collision cylinder length=0.12 radius=0.013; visual mesh filename=/home/user/unitree_ros2/cyclonedds_ws/src/dae/calf_mirror.d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
- link RR_foot: geometry collision sphere radius=0.022; visual mesh filename=/home/user/unitree_ros2/cyclonedds_ws/src/dae/foot.dae
- link RR_hip: geometry collision cylinder length=0.04 radius=0.046; visual mesh filename=/home/user/unitree_ros2/cyclonedds_ws/src/dae/hip.dae
- link RR_thigh: geometry collision box size=0.213 0.0245 0.034; visual mesh filename=/home/user/unitree_ros2/cyclonedds_ws/src/dae/thigh_mirror.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
- link base_link: geometry collision box size=0.3762 0.0935 0.114; visual mesh filename=/home/user/unitree_ros2/cyclonedds_ws/src/dae/base.dae

Commit message: move to jetson, change some files

File: cyclonedds_ws/src/urdf/go2.urdf (robot description, URDF)
Before this commit: robot go2, 31 links, 30 joints
Links:
- link FL_calf: geometry collision cylinder length=0.12 radius=0.012; visual mesh filename=/home/jetson/sobaka/sobaka_go2aka_go2/cyclonedds_ws/src/dae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
- link FL_foot: geometry collision sphere radius=0.022; visual mesh filename=/home/jetson/sobaka/sobaka_go2aka_go2/cyclonedds_ws/src/dae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
- link FL_hip: geometry collision cylinder length=0.04 radius=0.046; visual mesh filename=/home/jetson/sobaka/sobaka_go2/cyclonedds_ws/src/dae/hip.dae
- link FL_thigh: geometry collision box size=0.213 0.0245 0.034; visual mesh filename=/home/jetson/sobaka/sobaka_go2aka_go2/cyclonedds_ws/src/dae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
- link FR_calf: geometry collision cylinder length=0.12 radius=0.013; visual mesh filename=/home/jetson/sobaka/sobaka_go2/cyclonedds_ws/src/dae/calf_m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
- link FR_foot: geometry collision sphere radius=0.022; visual mesh filename=/home/jetson/sobaka/sobaka_go2/cyclonedds_ws/src/dae/foot.d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
- link FR_hip: geometry collision cylinder length=0.04 radius=0.046; visual mesh filename=/home/jetson/sobaka/sobaka_go2aka_go2/cyclonedds_ws/src/dae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
- link FR_thigh: geometry collision box size=0.213 0.0245 0.034; visual mesh filename=/home/jetson/sobaka/sobaka_go2/cyclonedds_ws/src/dae/thigh_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
- link RL_calf: geometry collision cylinder length=0.12 radius=0.013; visual mesh filename=/home/jetson/sobaka/sobaka_go2/cyclonedds_ws/src/dae/calf.d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
- link RL_foot: geometry collision sphere radius=0.022; visual mesh filename=/home/jetson/sobaka/sobaka_go2/cyclonedds_ws/src/dae/foot.d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
- link RL_hip: geometry collision cylinder length=0.04 radius=0.046; visual mesh filename=/home/jetson/sobaka/sobaka_go2/cyclonedds_ws/src/dae/hip.dae
- link RL_thigh: geometry collision box size=0.213 0.0245 0.034; visual mesh filename=/home/jetson/sobaka/sobaka_go2/cyclonedds_ws/src/dae/thigh.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
- link RR_calf: geometry collision cylinder length=0.12 radius=0.013; visual mesh filename=/home/jetson/sobaka/sobaka_go2/cyclonedds_ws/src/dae/calf_m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
- link RR_foot: geometry collision sphere radius=0.022; visual mesh filename=/home/jetson/sobaka/sobaka_go2/cyclonedds_ws/src/dae/foot.d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
- link RR_hip: geometry collision cylinder length=0.04 radius=0.046; visual mesh filename=/home/jetson/sobaka/sobaka_go2/cyclonedds_ws/src/dae/hip.dae
- link RR_thigh: geometry collision box size=0.213 0.0245 0.034; visual mesh filename=/home/jetson/sobaka/sobaka_go2/cyclonedds_ws/src/dae/thigh_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
- link base_link: geometry collision box size=0.3762 0.0935 0.114; visual mesh filename=/home/jetson/sobaka/sobaka_go2/cyclonedds_ws/src/dae/base.d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
